File: Bluelight/Bluelight.sch (EAGLE design)
At the start: 63 parts, among them J1 10118193-0001LF, J3 JST-2, J4 U.FL, J5 10118193-0001LF, U1 NRF51822, U2 ATSAMD21E18A-MUT, U3 TPS61200, U4 MCP73831, U5 TLV1117LV33, X1 16MHz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

Commit message: Fixing up keepout and part numbers.
Parts:
- C1, C10, C11, C12, C13, C14, C15, C2, C23, C24, C25, C28, C3, C4, C5, C6, C7, C8, C9: device Nordic:CAP-402 -> Nordic:CAP-0402
- C21, C22, C31: device Passives:CAP-402 -> Passives:CAP-0402
- L1, L2, L3, L5: device Nordic:IND-402 -> Nordic:IND-0402
- R11, R12, R2, R3, R4, R8: device Passives:RES-402 -> Passives:RES-0402
- R6: device Nordic:RES-402 -> Nordic:RES-0402
Changed lines of the file:
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@@
 <part name="SUPPLY3" library="SparkFun-Aesthetics" deviceset="3.3V" device=""/>
 <part name="SUPPLY4" library="SparkFun-Aesthetics" deviceset="3.3V" device=""/>
-<part name="C2" library="Nordic" deviceset="CAP-402" device="" value="47nF"/>
+<part name="C2" library="Nordic" deviceset="CAP-0402" device="" value="47nF"/>
 <part name="GND6" library="SparkFun-Aesthetics" deviceset="GND" device=""/>
-<part name="C3" library="Nordic" deviceset="CAP-402" device="" value="1nF"/>
+<part name="C3" library="Nordic" deviceset="CAP-0402" device="" value="1nF"/>
 <part name="GND7" library="SparkFun-Aesthetics" deviceset="GND" device=""/>
-<part name="C4" library="Nordic" deviceset="CAP-402" device="" value="100nF"/>
+<part name="C4" library="Nordic" deviceset="CAP-0402" device="" value="100nF"/>
 <part name="GND8" library="SparkFun-Aesthetics" deviceset="GND" device=""/>
-<part name="C5" library="Nordic" deviceset="CAP-402" device="" value="100nF"/>
+<part name="C5" library="Nordic" deviceset="CAP-0402" device="" value="100nF"/>
 <part name="GND9" library="SparkFun-Aesthetics" deviceset="GND" device=""/>
-<part name="C6" library="Nordic" deviceset="CAP-402" device="" value="100nF"/>
+<part name="C6" library="Nordic" deviceset="CAP-0402" device="" value="100nF"/>
 <part name="GND10" library="SparkFun-Aesthetics" deviceset="GND" device=""/>
-<part name="C7" library="Nordic" deviceset="CAP-402" device="" value="12pF"/>
-<part name="C8" library="Nordic" deviceset="CAP-402" device="" value="12pF"/>
+<part name="C7" library="Nordic" deviceset="CAP-0402" device="" value="12pF"/>
+<part name="C8" library="Nordic" deviceset="CAP-0402" device="" value="12pF"/>
 <part name="GND11" library="SparkFun-Aesthetics" deviceset="GND" device=""/>
 <part name="GND12" library="SparkFun-Aesthetics" deviceset="GND" device=""/>
@@
 <part name="X2" library="Nordic" deviceset="CRYSTAL" device="3215" value="32kHz"/>
 <part name="GND14" library="SparkFun-Aesthetics" deviceset="GND" device=""/>
-<part name="C9" library="Nordic" deviceset="CAP-402" device="" value="12pF"/>
-<part name="C10" library="Nordic" deviceset="CAP-402" device="" value="12pF"/>
+<part name="C9" library="Nordic" deviceset="CAP-0402" device="" value="12pF"/>
+<part name="C10" library="Nordic" deviceset="CAP-0402" device="" value="12pF"/>
 <part name="FRAME1" library="SparkFun-Aesthetics" deviceset="FRAME-LETTER" device="NO_PACKAGE"/>
 <part name="FRAME2" library="SparkFun-Aesthetics" deviceset="FRAME-LETTER" device="NO_PACKAGE"/>
 <part name="GND5" library="SparkFun-Aesthetics" deviceset="GND" device=""/>
-<part name="C1" library="Nordic" deviceset="CAP-402" device="" value="2.2nF"/>
-<part name="C11" library="Nordic" deviceset="CAP-402" device="" value="2.2pF"/>
-<part name="C12" library="Nordic" deviceset="CAP-402" device="" value="1.0pF"/>
-<part name="C13" library="Nordic" deviceset="CAP-402" device="" value="1.5pF"/>
+<part name="C1" library="Nordic" deviceset="CAP-0402" device="" value="2.2nF"/>
+<part name="C11" library="Nordic" deviceset="CAP-0402" device="" value="2.2pF"/>
+<part name="C12" library="Nordic" deviceset="CAP-0402" device="" value="1.0pF"/>
+<part name="C13" library="Nordic" deviceset="CAP-0402" device="" value="1.5pF"/>
 <part name="GND15" library="SparkFun-Aesthetics" deviceset="GND" device=""/>
 <part name="GND16" library="SparkFun-Aesthetics" deviceset="GND" device=""/>
-<part name="C14" library="Nordic" deviceset="CAP-402" device="" value="0pF"/>
-<part name="C15" library="Nordic" deviceset="CAP-402" device="" value="0pF"/>
+<part name="C14" library="Nordic" deviceset="CAP-0402" device="" value="0pF"/>
+<part name="C15" library="Nordic" deviceset="CAP-0402" device="" value="0pF"/>
 <part name="GND17" library="SparkFun-Aesthetics" deviceset="GND" device=""/>
 <part name="GND18" library="SparkFun-Aesthetics" deviceset="GND" device=""/>
-<part name="L5" library="Nordic" deviceset="IND-402" device="" value="4.7nH"/>
-<part name="L1" library="Nordic" deviceset="IND-402" device="" value="10nH"/>
-<part name="L2" library="Nordic" deviceset="IND-402" device="" value="3.3nH"/>
-<part name="L3" library="Nordic" deviceset="IND-402" device="" value="0nH"/>
+<part name="L5" library="Nordic" deviceset="IND-0402" device="" value="4.7nH"/>
+<part name="L1" library="Nordic" deviceset="IND-0402" device="" value="10nH"/>
+<part name="L2" library="Nordic" deviceset="IND-0402" device="" value="3.3nH"/>
+<part name="L3" library="Nordic" deviceset="IND-0402" device="" value="0nH"/>
 <part name="GND4" library="SparkFun-Aesthetics" deviceset="GND" device=""/>
 <part name="ANT1" library="Nordic" deviceset="MEANDER-ANT" device=""/>
@@
 <part name="GND40" library="SparkFun-Aesthetics" deviceset="GND" device=""/>
 <part name="GND41" library="SparkFun-Aesthetics" deviceset="GND" device=""/>
-<part name="C23" library="Nordic" deviceset="CAP-402" device="" value="4.7uF"/>
-<part name="C24" library="Nordic" deviceset="CAP-402" device="" value="4.7uF"/>
-<part name="R6" library="Nordic" deviceset="RES-402" device="" value="2k"/>
+<part name="C23" library="Nordic" deviceset="CAP-0402" device="" value="4.7uF"/>
+<part name="C24" library="Nordic" deviceset="CAP-0402" device="" value="4.7uF"/>
+<part name="R6" library="Nordic" deviceset="RES-0402" device="" value="2k"/>
 <part name="TC2" library="TagConnect" deviceset="TC2030-IDC" device="-NL"/>
 <part name="SUPPLY7" library="SparkFun-Aesthetics" deviceset="3.3V" device=""/>
@@
 <part name="C30" library="SparkFun-Passives" deviceset="CAP" device="1206" value="22uF"/>
 <part name="GND53" library="SparkFun-Aesthetics" deviceset="GND" device=""/>
-<part name="C21" library="Passives" deviceset="CAP-402" device="" value="0.1uF"/>
+<part name="C21" library="Passives" deviceset="CAP-0402" device="" value="0.1uF"/>
 <part name="GND26" library="SparkFun-Aesthetics" deviceset="GND" device=""/>
 <part name="R1" library="SparkFun-Passives" deviceset="RESISTOR" device="0805-RES" value="220k"/>
 <part name="R10" library="SparkFun-Passives" deviceset="RESISTOR" device="0805-RES" value="2M"/>
-<part name="C22" library="Passives" deviceset="CAP-402" device="" value="0.1uF"/>
+<part name="C22" library="Passives" deviceset="CAP-0402" device="" value="0.1uF"/>
 <part name="J3" library="SparkFun-Connectors" deviceset="JST_2MM_MALE" device="" value="JST-2"/>
 <part name="U2" library="atmel-samd21" deviceset="ATSAMD21E18A-MUT" device=""/>
-<part name="C25" library="Nordic" deviceset="CAP-402" device="" value="20pF"/>
-<part name="C28" library="Nordic" deviceset="CAP-402" device="" value="20pF"/>
+<part name="C25" library="Nordic" deviceset="CAP-0402" device="" value="20pF"/>
+<part name="C28" library="Nordic" deviceset="CAP-0402" device="" value="20pF"/>
 <part name="GND31" library="SparkFun-Aesthetics" deviceset="GND" device=""/>
 <part name="GND42" library="SparkFun-Aesthetics" deviceset="GND" device=""/>
@@
 <part name="GND44" library="SparkFun-Aesthetics" deviceset="GND" device=""/>
 <part name="GND54" library="SparkFun-Aesthetics" deviceset="GND" device=""/>
-<part name="C31" library="Passives" deviceset="CAP-402" device="" value="1uF"/>
+<part name="C31" library="Passives" deviceset="CAP-0402" device="" value="1uF"/>
 <part name="GND55" library="SparkFun-Aesthetics" deviceset="GND" device=""/>
 <part name="X4" library="Nordic" deviceset="CRYSTAL" device="3215" value="32kHz"/>
-<part name="R8" library="Passives" deviceset="RES-402" device="" value="100k"/>
-<part name="R11" library="Passives" deviceset="RES-402" device="" value="300k"/>
+<part name="R8" library="Passives" deviceset="RES-0402" device="" value="100k"/>
+<part name="R11" library="Passives" deviceset="RES-0402" device="" value="300k"/>
 <part name="GND2" library="SparkFun-Aesthetics" deviceset="GND" device=""/>
-<part name="R12" library="Passives" deviceset="RES-402" device="" value="4.7k"/>
+<part name="R12" library="Passives" deviceset="RES-0402" device="" value="4.7k"/>
 <part name="GND20" library="SparkFun-Aesthetics" deviceset="GND" device=""/>
 <part name="U$1" library="EVQ-PF206K" deviceset="EVQ-PF206K" device=""/>
@@
 <part name="GND22" library="SparkFun-Aesthetics" deviceset="GND" device=""/>
 <part name="D1" library="SparkFun-LED" deviceset="LED-RGB-CC-THRU" device="DIFFUSE"/>
-<part name="R2" library="Passives" deviceset="RES-402" device="" value="330"/>
-<part name="R3" library="Passives" deviceset="RES-402" device="" value="330"/>
-<part name="R4" library="Passives" deviceset="RES-402" device="" value="330"/>
+<part name="R2" library="Passives" deviceset="RES-0402" device="" value="330"/>
+<part name="R3" library="Passives" deviceset="RES-0402" device="" value="330"/>
+<part name="R4" library="Passives" deviceset="RES-0402" device="" value="330"/>
 <part name="J5" library="10118193-0001LF" deviceset="10118193-0001LF" device=""/>
 <part name="J1" library="10118193-0001LF" deviceset="10118193-0001LF" device=""/>
